Commit message: 4 camera sim

File: raspberry_ws/src/wizzybug_description/urdf/wizzybug.xacro (robot description, xacro)
@@ -253,8 +253,14 @@
     </joint>
     <link name="front_cam_link"/>
+    <joint name="front_cam_optical_joint" type="fixed">
+        <parent link="front_cam_link"/>
+        <child link="front_cam_link_optical"/>
+        <origin xyz="0 0 0" rpy="${-pi/2} 0 ${-pi/2}"/>
+    </joint>
+    <link name="front_cam_link_optical"/>
    <!-- <sensor_d415 parent="front_cam_link" name="camera1">
         <origin xyz="0 0 0" rpy="0 0 0"/>
-    </sensor_d415>
-        &lt;!&ndash; ################################ right cam ##############################################&ndash;&gt;
+    </sensor_d415>-->
+        <!-- ################################ right cam ##############################################-->
     <joint name="right_cam_joint" type="fixed">
         <parent link="base_link"/>
@@ -263,8 +269,14 @@
     </joint>
     <link name="right_cam_link"/>
-    <sensor_d415 parent="right_cam_link" name="camera2">
-        <origin xyz="0 0 0" rpy="0 0 0"/>
-    </sensor_d415>
-            &lt;!&ndash; ################################ left cam ##############################################&ndash;&gt;
+    <joint name="right_cam_optical_joint" type="fixed">
+        <parent link="right_cam_link"/>
+        <child link="right_cam_link_optical"/>
+        <origin xyz="0 0 0" rpy="${-pi/2} 0 ${-pi/2}"/>
+    </joint>
+    <link name="right_cam_link_optical"/>
+<!--    <sensor_d415 parent="right_cam_link" name="camera2">-->
+<!--        <origin xyz="0 0 0" rpy="0 0 0"/>-->
+<!--    </sensor_d415>-->
+<!--            &lt;!&ndash; ################################ left cam ##############################################&ndash;&gt;-->
     <joint name="left_cam_joint" type="fixed">
         <parent link="base_link"/>
@@ -273,8 +285,14 @@
     </joint>
     <link name="left_cam_link"/>
-    <sensor_d415 parent="left_cam_link" name="camera3">
-        <origin xyz="0 0 0" rpy="0 0 0"/>
-    </sensor_d415>
-                &lt;!&ndash; ################################ back cam ##############################################&ndash;&gt;
+    <joint name="left_cam_optical_joint" type="fixed">
+        <parent link="left_cam_link"/>
+        <child link="left_cam_link_optical"/>
+        <origin xyz="0 0 0" rpy="${-pi/2} 0 ${-pi/2}"/>
+    </joint>
+    <link name="left_cam_link_optical"/>
+<!--    <sensor_d415 parent="left_cam_link" name="camera3">-->
+<!--        <origin xyz="0 0 0" rpy="0 0 0"/>-->
+<!--    </sensor_d415>-->
+<!--                &lt;!&ndash; ################################ back cam ##############################################&ndash;&gt;-->
     <joint name="back_cam_joint" type="fixed">
         <parent link="base_link"/>
@@ -283,7 +301,13 @@
     </joint>
     <link name="back_cam_link"/>
-    <sensor_d415 parent="back_cam_link" name="camera4">
-        <origin xyz="0 0 0" rpy="0 0 0"/>
-    </sensor_d415>-->
+    <joint name="back_cam_optical_joint" type="fixed">
+        <parent link="back_cam_link"/>
+        <child link="back_cam_link_optical"/>
+        <origin xyz="0 0 0" rpy="${-pi/2} 0 ${-pi/2}"/>
+    </joint>
+    <link name="back_cam_link_optical"/>
+<!--    <sensor_d415 parent="back_cam_link" name="camera4">-->
+<!--        <origin xyz="0 0 0" rpy="0 0 0"/>-->
+<!--    </sensor_d415>&ndash;&gt;-->
     <!-- ################################ rplidar ##############################################-->
     <joint name="rplidar_joint" type="fixed">

Commit message: renamed back_camera to rear_camera. starting to configure multiple cameras

File: raspberry_ws/src/wizzybug_description/urdf/wizzybug.xacro (robot description, xacro)
@@ -31,7 +31,7 @@
     <xacro:property name="right_cam_y" value="-0.26"/>
     <xacro:property name="right_cam_z" value="0.16"/>
-    <xacro:property name="back_cam_x" value="-0.48"/>
-    <xacro:property name="back_cam_y" value="0.0"/>
-    <xacro:property name="back_cam_z" value="0.63"/>
+    <xacro:property name="rear_cam_x" value="-0.48"/>
+    <xacro:property name="rear_cam_y" value="0.0"/>
+    <xacro:property name="rear_cam_z" value="0.63"/>
     <xacro:property name="rplidar_x" value="0.0"/>
     <xacro:property name="rplidar_y" value="0.1"/>
@@ -294,18 +294,18 @@
 <!--        <origin xyz="0 0 0" rpy="0 0 0"/>-->
 <!--    </sensor_d415>-->
-<!--                &lt;!&ndash; ################################ back cam ##############################################&ndash;&gt;-->
-    <joint name="back_cam_joint" type="fixed">
-        <parent link="base_link"/>
-        <child link="back_cam_link"/>
-        <origin xyz="${back_cam_x} 0 ${back_cam_z}" rpy="0 0 3.14"/>
-    </joint>
-    <link name="back_cam_link"/>
-    <joint name="back_cam_optical_joint" type="fixed">
-        <parent link="back_cam_link"/>
-        <child link="back_cam_link_optical"/>
+<!--                &lt;!&ndash; ################################ rear cam ##############################################&ndash;&gt;-->
+    <joint name="rear_cam_joint" type="fixed">
+        <parent link="base_link"/>
+        <child link="rear_cam_link"/>
+        <origin xyz="${rear_cam_x} 0 ${rear_cam_z}" rpy="0 0 3.14"/>
+    </joint>
+    <link name="rear_cam_link"/>
+    <joint name="rear_cam_optical_joint" type="fixed">
+        <parent link="rear_cam_link"/>
+        <child link="rear_cam_link_optical"/>
         <origin xyz="0 0 0" rpy="${-pi/2} 0 ${-pi/2}"/>
     </joint>
-    <link name="back_cam_link_optical"/>
-<!--    <sensor_d415 parent="back_cam_link" name="camera4">-->
+    <link name="rear_cam_link_optical"/>
+<!--    <sensor_d415 parent="rear_cam_link" name="camera4">-->
 <!--        <origin xyz="0 0 0" rpy="0 0 0"/>-->
 <!--    </sensor_d415>&ndash;&gt;-->
