Commit message: before going into vision related aspects

File: src/common/wizzybug_description/urdf/wizzybug.xacro (robot description, xacro)
@@ -143,10 +143,9 @@
         </inertial>
     </link>
-    <joint name="left_caster_axle_joint" type="continuous">
+    <joint name="left_caster_axle_joint" type="fixed">
         <parent link="base_link"/>
         <child link="left_caster_axle_link"/>
         <origin xyz="${-caster_axis_x}  ${caster_wheel_base/2+wheel_thickness/2} ${caster_axis_z}" rpy="0 0 0"/>
-        <axis xyz="0 0 1"/>
-        <dynamics damping="${caster_damping}" friction="${caster_friction}"/>
+        <!-- <dynamics damping="${caster_damping}" friction="${caster_friction}"/> -->
     </joint>
     <link name="left_caster_link">
@@ -173,5 +172,4 @@
         </inertial>
     </link>
-<!--
     <joint name="left_caster_joint" type="continuous">
         <parent link="left_caster_axle_link"/>
@@ -181,5 +179,5 @@
         <dynamics damping="${wheel_damping}" friction="${wheel_friction}"/>
     </joint>
--->
+<!--
     <joint name="left_caster_joint" type="continuous">
         <parent link="base_link"/>
@@ -189,4 +187,5 @@
         <dynamics damping="${wheel_damping}" friction="${wheel_friction}"/>
     </joint>
+-->
     <!-- ################################Right caster Wheel##############################################-->
     <link name="right_caster_axle_link">
@@ -200,10 +199,9 @@
         </inertial>
     </link>
-    <joint name="right_caster_axle_joint" type="continuous">
+    <joint name="right_caster_axle_joint" type="fixed">
         <parent link="base_link"/>
         <child link="right_caster_axle_link"/>
         <origin xyz="${-caster_axis_x} ${-caster_wheel_base/2-wheel_thickness/2} ${caster_axis_z}" rpy="0 0 0"/>
-        <axis xyz="0 0 1"/>
-        <dynamics damping="${caster_damping}" friction="${caster_friction}"/>
+        <!-- <dynamics damping="${caster_damping}" friction="${caster_friction}"/> -->
     </joint>
     <link name="right_caster_link">
@@ -230,5 +228,4 @@
         </inertial>
     </link>
-<!--
     <joint name="right_caster_joint" type="continuous">
         <parent link="right_caster_axle_link"/>
@@ -238,5 +235,5 @@
         <dynamics damping="${wheel_damping}" friction="${wheel_friction}"/>
     </joint>
--->
+<!--
     <joint name="right_caster_joint" type="continuous">
         <parent link="base_link"/>
@@ -246,4 +243,5 @@
         <dynamics damping="${wheel_damping}" friction="${wheel_friction}"/>
     </joint>
+-->
     <!-- ################################imu##############################################-->
     <link name="imu_link"/>
@@ -306,5 +304,5 @@
 <!--        <origin xyz="0 0 0" rpy="0 0 0"/>-->
 <!--    </sensor_d415>-->
-<!--            &lt;!&ndash; ################################ left cam ##############################################&ndash;&gt;-->
+<!--  ################################ left cam ############################################## -->
     <joint name="left_cam_joint" type="fixed">
         <parent link="base_link"/>
@@ -322,5 +320,5 @@
 <!--        <origin xyz="0 0 0" rpy="0 0 0"/>-->
 <!--    </sensor_d415>-->
-<!--                &lt;!&ndash; ################################ rear cam ##############################################&ndash;&gt;-->
+<!-- ################################ rear cam ##############################################-->
     <joint name="rear_cam_joint" type="fixed">
         <parent link="base_link"/>

Commit message: preliminary working position-based decision maker with simulated obstacles

File: src/common/wizzybug_description/urdf/wizzybug.xacro (robot description, xacro)
@@ -21,4 +21,5 @@
     <xacro:property name="caster_damping" value="0.0"/>
     <xacro:property name="wheel_mass" value="1.0"/>
+    <xacro:property name="tire_friction" value="1.0"/>
     <xacro:property name="caster_wheel_base" value="0.32"/>
     <xacro:property name="caster_axis_x" value="0.45"/>
@@ -79,4 +80,12 @@
             <material name="black"/>
         </visual>
+        <surface>
+            <friction>
+                  <ode>
+                        <slip1>"${tire_friction}"</slip1>
+                        <slip2>"${tire_friction}"</slip2>
+                  </ode>
+            </friction>
+        </surface>
         <collision>
             <geometry>
@@ -110,4 +119,12 @@
             <material name="black"/>
         </visual>
+        <surface>
+            <friction>
+                  <ode>
+                        <slip1>"${tire_friction}"</slip1>
+                        <slip2>"${tire_friction}"</slip2>
+                  </ode>
+            </friction>
+        </surface>
         <collision>
             <geometry>
@@ -157,4 +174,12 @@
             <material name="black"/>
         </visual>
+        <surface>
+            <friction>
+                  <ode>
+                        <slip1>"${tire_friction}"</slip1>
+                        <slip2>"${tire_friction}"</slip2>
+                  </ode>
+            </friction>
+        </surface>
         <collision>
             <geometry>
@@ -213,4 +238,12 @@
             <material name="black"/>
         </visual>
+        <surface>
+            <friction>
+                  <ode>
+                        <slip1>"${tire_friction}"</slip1>
+                        <slip2>"${tire_friction}"</slip2>
+                  </ode>
+            </friction>
+        </surface>
         <collision>
             <geometry>

Commit message: layed foundation for lidar testing

File: src/common/wizzybug_description/urdf/wizzybug.xacro (robot description, xacro)
@@ -21,5 +21,4 @@
     <xacro:property name="caster_damping" value="0.0"/>
     <xacro:property name="wheel_mass" value="1.0"/>
-    <xacro:property name="tire_friction" value="1.0"/>
     <xacro:property name="caster_wheel_base" value="0.32"/>
     <xacro:property name="caster_axis_x" value="0.45"/>
@@ -80,12 +79,4 @@
             <material name="black"/>
         </visual>
-        <surface>
-            <friction>
-                  <ode>
-                        <slip1>"${tire_friction}"</slip1>
-                        <slip2>"${tire_friction}"</slip2>
-                  </ode>
-            </friction>
-        </surface>
         <collision>
             <geometry>
@@ -119,12 +110,4 @@
             <material name="black"/>
         </visual>
-        <surface>
-            <friction>
-                  <ode>
-                        <slip1>"${tire_friction}"</slip1>
-                        <slip2>"${tire_friction}"</slip2>
-                  </ode>
-            </friction>
-        </surface>
         <collision>
             <geometry>
@@ -174,12 +157,4 @@
             <material name="black"/>
         </visual>
-        <surface>
-            <friction>
-                  <ode>
-                        <slip1>"${tire_friction}"</slip1>
-                        <slip2>"${tire_friction}"</slip2>
-                  </ode>
-            </friction>
-        </surface>
         <collision>
             <geometry>
@@ -238,12 +213,4 @@
             <material name="black"/>
         </visual>
-        <surface>
-            <friction>
-                  <ode>
-                        <slip1>"${tire_friction}"</slip1>
-                        <slip2>"${tire_friction}"</slip2>
-                  </ode>
-            </friction>
-        </surface>
         <collision>
             <geometry>

Commit message: before testing on wizzy for the first time

File: src/common/wizzybug_description/urdf/wizzybug.xacro (robot description, xacro)
@@ -40,5 +40,5 @@
     <xacro:property name="rplidar_x" value="0.1"/>
     <xacro:property name="rplidar_y" value="0.1"/>
-    <xacro:property name="rplidar_z" value="0.0"/>
+    <xacro:property name="rplidar_z" value="0.05"/>
     <link name="base_footprint">
     </link>
@@ -340,5 +340,5 @@
         <parent link="base_link"/>
         <child link="rplidar_link"/>
-        <origin xyz="${rplidar_x} ${rplidar_y} ${rplidar_z}" rpy="1.5708 0 0"/>
+        <origin xyz="${rplidar_x} ${rplidar_y} ${rplidar_z}" rpy="1.5708 1.45 0"/>
     </joint>
     <link name="rplidar_link">
@@ -361,3 +361,27 @@
         </inertial>
     </link>
+    <joint name="laser_joint" type="fixed">
+        <parent link="base_link"/>
+        <child link="laser"/>
+        <origin xyz="${rplidar_x} ${rplidar_y} ${rplidar_z}" rpy="1.5708 1.45 0"/>
+    </joint>
+    <link name="laser">
+        <collision>
+            <origin xyz="0 0 0" rpy="0 0 0"/>
+            <geometry>
+            <cylinder length="0.05" radius="0.025"/>
+            </geometry>
+        </collision>
+        <visual>
+            <origin xyz="0 0 0" rpy="0 0 0"/>
+            <geometry>
+            <cylinder length="0.05" radius="0.025"/>
+            </geometry>
+        </visual>
+        <inertial>
+            <mass value="1e-5"/>
+            <origin xyz="0 0 0" rpy="0 0 0"/>
+            <inertia ixx="1e-6" ixy="0" ixz="0" iyy="1e-6" iyz="0" izz="1e-6"/>
+        </inertial>
+    </link>
 </robot>
